File: adsr2.brd (EAGLE design)
At the start: 99.4 x 29.2 mm, 57 parts, among them IC1 LM324D, IC2 4066D, IC3 4555D, SW1_TIME TL2285 L, SW2_TRIG TL2285 L, T1 BC847, T2 BC857, T3 BC857, T4 BC847, T5 BC857

Commit message: Changed some resistors from 100k to 10k; this works with the used BC847 transistors. (Breadboard prototype used BC547B)
Parts:
- R20, R25, R7, R9: value 100k -> 10k
Changed lines of the file:
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@@
 </element>
 <element name="R2" library="pot-alps" package="ALPS_POT_VERTICAL" value="100k" x="58.42" y="30.48" rot="MR270"/>
-<element name="R20" library="rcl" package="R0603" value="100k" x="13.335" y="18.415" smashed="yes">
+<element name="R20" library="rcl" package="R0603" value="10k" x="13.335" y="18.415" smashed="yes">
 <attribute name="NAME" x="12.065" y="16.51" size="0.8128" layer="25" font="vector"/>
 </element>
@@
 <element name="R4" library="pot-alps" package="ALPS_POT_VERTICAL" value="1M" x="76.2" y="30.48" rot="MR270"/>
 <element name="R5" library="pot-alps" package="ALPS_POT_VERTICAL" value="1M" x="93.98" y="30.48" rot="MR270"/>
-<element name="R9" library="rcl" package="R0603" value="100k" x="12.7" y="24.765" smashed="yes">
+<element name="R9" library="rcl" package="R0603" value="10k" x="12.7" y="24.765" smashed="yes">
 <attribute name="NAME" x="11.43" y="26.035" size="0.8128" layer="25" font="vector"/>
 </element>
@@
 <attribute name="NAME" x="79.64" y="31.01" size="0.8128" layer="25" font="vector" rot="R270"/>
 </element>
-<element name="R7" library="rcl" package="R0603" value="100k" x="6.985" y="23.495" smashed="yes" rot="R180">
+<element name="R7" library="rcl" package="R0603" value="10k" x="6.985" y="23.495" smashed="yes" rot="R180">
 <attribute name="NAME" x="7.62" y="22.225" size="0.8128" layer="25" font="vector" rot="R180"/>
 </element>
@@
 <attribute name="NAME" x="29.591" y="31.75" size="1.27" layer="26" ratio="10" rot="MR90"/>
 </element>
-<element name="R25" library="rcl" package="R0603" value="100k" x="13.335" y="35.56" smashed="yes" rot="R270">
+<element name="R25" library="rcl" package="R0603" value="10k" x="13.335" y="35.56" smashed="yes" rot="R270">
 <attribute name="NAME" x="12.065" y="34.925" size="0.8128" layer="25" font="vector" rot="R90"/>
 </element>
