File: adsr_v3.sch (EAGLE design)
At the start: 48 parts, among them IC1 LM324D, IC2 4052D, IC3 40106D, SW1_TIME TL2285 L, SW2_TRIG TL2285 L, T1 BC847

Commit message: Minor routing & labeling fixes. Replaced schematic A3 document frame with other type.
Other:
- note added: "Attack"
- note added: "Decay"
- note added: "Release"
- note added: "Sustain Level"
Changed lines of the file:
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@@
 <text x="45.72" y="233.68" size="1.778" layer="91">TL2285 momentary
 Manual trigger button</text>
+<text x="91.44" y="114.3" size="1.778" layer="91">Attack</text>
+<text x="91.44" y="139.7" size="1.778" layer="91">Release</text>
+<text x="91.44" y="88.9" size="1.778" layer="91">Decay</text>
+<text x="20.32" y="93.98" size="1.778" layer="91">Sustain
+Level</text>
 </plain>
 <instances>

Commit message: Changed LED current resistors to 27k, better match with the 350-400 mcd LEDs.
Parts:
- R10, R24: value 10k -> 27k
Changed lines of the file:
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@@
 <part name="R9" library="rcl" deviceset="R-EU_" device="R0603" value="100k"/>
 <part name="T1" library="transistor" deviceset="BC847" device=""/>
-<part name="R10" library="rcl" deviceset="R-EU_" device="R0603" value="10k"/>
+<part name="R10" library="rcl" deviceset="R-EU_" device="R0603" value="27k"/>
 <part name="GND13" library="supply1" deviceset="GND" device=""/>
 <part name="GND14" library="supply1" deviceset="GND" device=""/>
@@
 <part name="R16" library="rcl" deviceset="R-EU_" device="R0603" value="3k3"/>
 <part name="GND10" library="supply1" deviceset="GND" device=""/>
-<part name="R24" library="rcl" deviceset="R-EU_" device="R0603" value="10k"/>
+<part name="R24" library="rcl" deviceset="R-EU_" device="R0603" value="27k"/>
 <part name="LED1" library="led" deviceset="LED" device="5MM" value="PEAK_LED"/>
 <part name="P+10" library="supply1" deviceset="+12V" device=""/>
